Commit message: initial implementation

File: src/abb/abb_irb2400_support/urdf/irb2400.urdf (robot description, URDF)
Before this commit: robot abb_irb2400, 9 links, 8 joints
Links:
- removed link base
- added link chassis; collision mesh filename=package://abb_irb2400_support/meshes/irb2400/collision/mobi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; visual mesh filename=package://abb_irb2400_support/meshes/irb2400/visual/mobile_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
- added link dummy
- added link left_back_wheel; collision mesh filename=package://abb_irb2400_support/meshes/irb2400/collision/whee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; visual mesh filename=package://abb_irb2400_support/meshes/irb2400/visual/wheel_m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
- added link left_front_wheel; collision mesh filename=package://abb_irb2400_support/meshes/irb2400/collision/whee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; visual mesh filename=package://abb_irb2400_support/meshes/irb2400/visual/wheel_m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
- added link right_back_wheel; collision mesh filename=package://abb_irb2400_support/meshes/irb2400/collision/whee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; visual mesh filename=package://abb_irb2400_support/meshes/irb2400/visual/wheel_m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
- added link right_front_wheel; collision mesh filename=package://abb_irb2400_support/meshes/irb2400/collision/whee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; visual mesh filename=package://abb_irb2400_support/meshes/irb2400/visual/wheel_m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
- added link suction_cup_end_effector; collision mesh filename=package://abb_irb2400_support/meshes/irb2400/collision/suct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; visual mesh filename=package://abb_irb2400_support/meshes/irb2400/visual/suction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
Joints:
- removed joint base_link-base
- added joint chassis_to_base_link: type fixed, parent chassis, child base_link, origin xyz=-0.2 0 0 rpy=0 0 0
- added joint dummy_joint: type fixed, parent dummy, child chassis, origin xyz=0.0 0.0 0.43 rpy=0 0 0
- added joint left_back_wheel_joint: type continuous, parent chassis, child right_front_wheel, origin xyz=0.465 -0.76 -0.35 rpy=0 0 0, axis 0 1 0, limit effort=100 velocity=100
- added joint left_front_wheel_joint: type continuous, parent chassis, child right_back_wheel, origin xyz=-0.535 -0.76 -0.35 rpy=0 0 0, axis 0 1 0, limit effort=100 velocity=100
- added joint right_back_wheel_joint: type continuous, parent chassis, child left_front_wheel, origin xyz=0.465 0.64 -0.35 rpy=0 0 0, axis 0 1 0, limit effort=100 velocity=100
- added joint right_front_wheel_joint: type continuous, parent chassis, child left_back_wheel, origin xyz=-0.535 0.64 -0.35 rpy=0 0 0, axis 0 1 0, limit effort=100 velocity=100
- added joint suction_to_tool0: type fixed, parent tool0, child suction_cup_end_effector, origin xyz=0 0 0 rpy=0 0 0

File: src/abb/abb_irb2400_support/urdf/irb2400_macro.xacro (robot description, xacro)
@@ -116,4 +116,21 @@
     </link>
     <link name="${prefix}tool0"/>
+<!--   Suction Cup   -->
+    <link name="${prefix}suction_cup_end_effector">
+        <visual>
+            <origin xyz="0 0 0.001" rpy="0 0 0"/>
+            <geometry>
+                <mesh filename="package://abb_irb2400_support/meshes/irb2400/visual/suction_cup.dae" />
+            </geometry>
+            <xacro:material_abb_leaf_green />
+        </visual>
+        <collision>
+            <origin xyz="0 0 0" rpy="0 0 0"/>
+            <geometry>
+                <mesh filename="package://abb_irb2400_support/meshes/irb2400/collision/suction_cup.stl" />
+            </geometry>
+            <xacro:material_abb_yellow />
+        </collision>
+    </link>
     <!-- end of link list -->
     <!-- joint list -->
@@ -165,12 +182,97 @@
         <origin xyz="0 0 0" rpy="0 1.57079632679 0"/>
     </joint>
+    <joint name="${prefix}tool0-suction_cup" type="fixed">
+        <parent link="${prefix}tool0"/>
+        <child link="${prefix}suction_cup_end_effector"/>
+        <origin xyz="0 0 0" rpy="0 0 0"/>
+    </joint>
     <!-- end of joint list -->
-    <!-- ROS base_link to ABB World Coordinates transform -->
-    <link name="${prefix}base" />
-    <joint name="${prefix}base_link-base" type="fixed">
-        <origin xyz="0 0 0" rpy="0 0 0"/>
-        <parent link="${prefix}base_link"/>
-        <child link="${prefix}base"/>
+<!--///////////////////////////////////////////////////////////////////////-->
+    <!--    Transmission Block-->
+    <xacro:macro name="Transmission_Block" params="joint_name">
+        <transmission name="${joint_name}_trans">
+            <type>transmission_interface/SimpleTransmission</type>
+            <joint name="${joint_name}">
+                <hardwareInterface>hardware_interface/PositionJointInterface</hardwareInterface>
+            </joint>
+            <actuator name="${joint_name}_motor">
+                <mechanicalReduction>1</mechanicalReduction>
+            </actuator>
+        </transmission>
+    </xacro:macro>
+    <!--    //////////////////////////////////////////////////////////////////////-->
+    <!--Dummy link-->
+    <link name="dummy"/>
+    <!--    Chassis-->
+    <link name = "chassis">
+        <visual>
+            <origin rpy = "3.14 0 0" xyz = "0 0 0"/>
+            <geometry>
+                <mesh filename="package://abb_irb2400_support/meshes/irb2400/visual/mobile_base.dae" />
+            </geometry>
+        </visual>
+        <collision>
+            <origin rpy = "3.14 0 0" xyz = "0 0 0"/>
+            <geometry>
+                <mesh filename="package://abb_irb2400_support/meshes/irb2400/collision/mobile_base.stl" />            </geometry>
+        </collision>
+    </link>
+    <joint name="dummy_joint" type="fixed">
+        <parent link="dummy"/>
+        <child link="chassis"/>
+        <origin xyz="0.0 0.0 0.43" rpy="0 0 0" />
+    </joint>
+    <!--    Wheels-->
+    <xacro:macro name="wheel" params="prefix suffix X Y Z">
+        <link name="${prefix}_${suffix}_wheel">
+            <visual>
+                <origin rpy="1.57 0 0" xyz="0 0 0"/>
+                <geometry>
+                    <mesh filename="package://abb_irb2400_support/meshes/irb2400/visual/wheel_mobile_base.dae" />
+                </geometry>
+                <material name="Black"/>
+            </visual>
+            <collision>
+                <origin rpy="1.57 0 0" xyz="0 0 0"/>
+                <geometry>
+                    <mesh filename="package://abb_irb2400_support/meshes/irb2400/collision/wheel_mobile_base.stl" />
+                </geometry>
+            </collision>
+        </link>>
+        <joint name="${prefix}_${suffix}_wheel_joint" type="continuous">
+            <parent link="chassis"/>
+            <child link="${prefix}_${suffix}_wheel"/>
+            <origin xyz="${X} ${Y} ${Z}" rpy="0 0 0"/>
+            <axis xyz="0 1 0"/>
+            <limit effort = "100" velocity = "100"/>
+            <dynamics damping = "0.0" friction = "0.0"/>
+        </joint>
+        <transmission name="${prefix}_${suffix}_wheel_trans">
+            <type>transmission_interface/SimpleTransmission</type>
+            <actuator name="${prefix}_${suffix}_wheel_motor">
+                <hardwareInterface>hardware_interface/VelocityJointInterface</hardwareInterface>
+                <mechanicalReduction>1</mechanicalReduction>
+            </actuator>
+            <joint name="${prefix}_${suffix}_wheel_joint">
+                <hardwareInterface>hardware_interface/VelocityJointInterface</hardwareInterface>
+            </joint>
+        </transmission>
+    </xacro:macro>
+    <xacro:wheel prefix="left" suffix="back" X="0.465" Y="-0.76" Z="-0.35"/>
+    <xacro:wheel prefix="left" suffix="front" X="-0.535" Y="-0.76" Z="-0.35"/>
+    <xacro:wheel prefix="right" suffix="back" X="0.465" Y="0.64" Z="-0.35"/>
+    <xacro:wheel prefix="right" suffix="front" X="-0.535" Y="0.64" Z="-0.35"/>
+    <!-- ROS base_link to mobile base Coordinates transform -->
+    <joint name="chassis_to_base_link" type="fixed">
+        <origin rpy="0 0 0" xyz="0 0 0"/>
+        <parent link="chassis"/>
+        <child link="${prefix}base_link"/>
     </joint>
 </xacro:macro>
+    <gazebo>
+        <plugin name="gazebo_ros_control"  filename="libgazebo_ros_control.so">
+            <robotNamespace>/</robotNamespace>
+            <legacyModeNS>true</legacyModeNS>
+        </plugin>
+    </gazebo>
 </robot>
